File: Laser Module/Mouse.brd (EAGLE design)
At the start: 100 x 40 mm, 85 parts, among them Q1 MOSFET-NCHANNELAO3404A, U1 RFM69HCW, U2 HALL-EFFECTSMD, U3 HALL-EFFECTSMD, U4 HALL-EFFECTSMD, U5 HALL-EFFECTSMD, U6 BQ27441-G1, U7 BQ24075, U8 ATSAMD21G-A, U9 3.3V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

Commit message: ACTUALLY finalized all of the PCBs and created .zip's containing the gerber files of each
Routing:
- net BATTERY_IN: track 20.2 -> 19.3 mm
