File: Dongle Module/Dongle.brd (EAGLE design)
At the start: 45 x 28 mm, 31 parts, among them Q2 2.5A/30V, U1 RFM69HCW, U10 74AHC1G125, U8 ATSAMD21G-A, U9 3.3V, Y1 32.768kHz

Commit message: push ui.c again
Parts:
- removed U$2: (no value), MAAV_BlockM:BLOCK-M-5MM
- removed U$4: (no value), MAAV_BlockM:BLOCK-M-10MM-MASK
- C12, C13, C14, C15: device SparkFun-Capacitors:0603-CAP -> SparkFun-Capacitors:0402-CAP
- C16, C17: device SparkFun-Capacitors:0603-CAP -> samd21-temp:0402-CAP
- C2: device SparkFun-Capacitors:0603-CAP -> SparkFun-Capacitors:0603-CAP@1
- D7: value GREEN -> RED
- moved C16 1.99 mm to (38.4, 3.89)
- moved C17 1.60 mm to (39.2, 7.10)
- moved Y1 1.10 mm to (41.9, 5.38)
- moved C13 0.45 mm to (33.8, 2.23)
- moved C15 0.40 mm to (26.2, 5.22)
- moved C12 0.36 mm to (34.2, 15.3)
- moved JP23 0.15 mm to (44.0, 14.0)
Routing:
- net RF_INT: track 46.0 -> 0.00 mm, vias 3 -> 0
- net N$13: track 6.21 -> 5.09 mm
- net N$10: track 6.85 -> 5.78 mm
- net USB_HOST_EN: track 37.2 -> 38.0 mm
- net 3.3V: track 91.4 -> 90.6 mm
- net GND: track 9.57 -> 10.2 mm
- net RF_SS: track 25.3 -> 24.7 mm
Other:
- board text removed: "AIZER"
- board text removed: "Designed By: Matt Sauvé"
- board text removed: "Dongle Module"
